Commit message: added Lidar, Camera and SLAM

File: description/depth_camera.xacro (robot description, xacro)
@@ -4,5 +4,5 @@
         <parent link="chassis"/>
         <child link="camera_link"/>
-        <origin xyz="0.305 0 0.08" rpy="0 0.18 0"/>
+        <origin xyz="0.305 0 0.08" rpy="0 0 0"/>
     </joint>
     <link name="camera_link">
@@ -22,5 +22,5 @@
     <gazebo reference="camera_link">
         <material>Gazebo/Red</material>
-        <sensor name="camera" type="camera">
+        <sensor name="camera" type="depth">
             <pose> 0 0 0 0 0 0 </pose>
             <visualize>true</visualize>
@@ -29,5 +29,5 @@
                 <horizontal_fov>1.089</horizontal_fov>
                 <image>
-                    <format>R8G8B8</format>
+                    <format>B8G8R8</format>
                     <width>640</width>
                     <height>480</height>
@@ -40,4 +40,6 @@
             <plugin name="camera_controller" filename="libgazebo_ros_camera.so">
                 <frame_name>camera_link_optical</frame_name>
+                <min_depth>0.1</min_depth>
+                <max_depth>100.0</max_depth>
             </plugin>
         </sensor>

File: description/robot.urdf.xacro (robot description, xacro)
@@ -3,6 +3,8 @@
     <!-- Example link -->
     <xacro:include filename="robot_core.xacro" />
-    <xacro:include filename="gazebo_control.xacro"/>
+    <!-- <xacro:include filename="gazebo_control.xacro"/> -->
+    <xacro:include filename="ros2_control.xacro"/>
     <xacro:include filename="lidar.xacro"/>
     <xacro:include filename="camera.xacro"/>
+    <!-- <xacro:include filename="depth_camera.xacro"/> -->
 </robot>

File: description/robot_core.xacro (robot description, xacro)
@@ -20,4 +20,11 @@
     <link name="base_link">
     </link>
+    <!-- BASE FOOTPRINT -->
+    <joint name="base_footprint_joint" type="fixed">
+        <parent link="base_link"/>
+        <child link= "base_footprint"/>
+        <origin xyz="0 0 0" rpy="0 0 0"/>
+    </joint>
+    <link name="base_footprint"></link>
     <!-- CHASSIS LINK -->
     <joint name="chassis_joint" type="fixed">
